File: 8086-processor.sch (KiCad schematic (older format))
At the start: 24 parts

Commit message: Replaced MWTC MRDC IOWC IORC with WR RD; buffered control bus; consolidated logic gates
Parts:
- removed U? (x5): 74LS32, symbol 74xx:74LS32
- removed U? (x3): 74LS14, symbol 74xx:74LS14
- added C?: 100nF, symbol Device:C
- added R?: 1k, symbol Device:R
- added U?: 74LS244, symbol 74xx:74LS244
Connections:
- net GND: now also C?.1, U?.1 (OEa), U?.10 (GND), U?.11 (I0b), U?.13 (I1b), U?.15 (I2b), U?.17 (I3b), U?.19 (OEb)
- net M\~IO: now also U?.18 (O0a); no longer U?.28 (M/~IO~)
- net NMI: now also U?.12 (O3a)
- net VCC: now also C?.2, R?.1, U?.20 (VCC); no longer U?.33 (MN/~MX~)
- net at U?.29 (~WR~): now also U?.4 (I1a)
- net at U?.32 (~RD~): now also U?.6 (I2a)
- net at C?.1, R?.1: now also U?.8 (I3a)
- new net: U?.2 (I0a), U?.28 (M/~IO~)
- new net: R?.2, U?.33 (MN/~MX~)
- new net ~RD: U?.14 (O2a)
- new net ~WR: U?.16 (O1a)
- no-connect marks 6 -> 10
Other:
- note removed: "Memory-/IO-\nRead/Write\nSignal Decoding"
