File: CMOS-flash.sch (KiCad schematic (older format))
At the start: 10 parts

Commit message: Replaced MWTC MRDC IOWC IORC with WR RD; buffered control bus; consolidated logic gates
Connections:
- net ~MRDC renamed ~RD
- net ~MWTC renamed ~WR
Changed lines of the file:
@@
 $Descr A4 11693 8268
 encoding utf-8
-Sheet 5 10
+Sheet 4 11
 Title "CMOS-flash"
 Date ""
@@
 $EndComp
 Text HLabel 8300 1950 2    50   Input ~ 0
-~MWTC
+~WR
 Text HLabel 8300 4400 2    50   Input ~ 0
-~MWTC
+~WR
 Text HLabel 8300 5100 2    50   Input ~ 0
-~MRDC
+~RD
 Text HLabel 8300 2650 2    50   Input ~ 0
-~MRDC
+~RD
 NoConn ~ 8300 2050
 NoConn ~ 8300 4500
