File: CMOS-flash.sch (KiCad schematic (older format))
At the start: 10 parts

Commit message: Updates to pass ERC
Changed lines of the file:
@@
 	6000 5700 5900 5800
 Text HLabel 5900 5900 0    50   BiDi ~ 0
-DATA_BUS
+D[0..15]
 Text HLabel 8500 6000 2    50   BiDi ~ 0
-DATA_BUS
+D[0..15]
 Entry Wire Line
 	8700 2250 8800 2150
@@
 	8700 2750 8300 2750
 Text HLabel 8800 1950 2    50   Input ~ 0
-ADDRESS_BUS
+A[0..19]
 Entry Wire Line
 	5750 1950 5650 1850
@@
 	6100 2950 5750 2950
 Text HLabel 8550 3600 2    50   BiDi ~ 0
-DATA_BUS
+D[0..15]
 Text HLabel 5850 3450 0    50   BiDi ~ 0
-DATA_BUS
+D[0..15]
 Text Label 5750 2950 0    50   ~ 0
 A1
@@
 	8700 5200 8300 5200
 Text HLabel 8800 4400 2    50   Input ~ 0
-ADDRESS_BUS
+A[0..19]
 Text Label 8700 5200 2    50   ~ 0
 A11
@@
 	6100 5400 5750 5400
 Text HLabel 5650 4200 0    50   Input ~ 0
-ADDRESS_BUS
+A[0..19]
 Text Label 5750 5400 0    50   ~ 0
 A1
@@
 A19
 Text HLabel 1400 2600 2    50   Input ~ 0
-ADDRESS_BUS
+A[0..19]
 Text HLabel 5650 1750 0    50   Input ~ 0
-ADDRESS_BUS
+A[0..19]
 Text Label 3500 3100 0    50   ~ 0
 ~CE_HI_BYTE

Commit message: Assign footprints for most symbols
Parts:
- C29, C30, C31, C32, C33, C34: renamed from C?; footprint (none) -> Capacitor_THT:C_Rect_L4.0mm_W2.5mm_P2.50mm
- U25, U26: renamed from U?; footprint (none) -> Package_DIP:DIP-20_W7.62mm
- U27, U28: renamed from U?; footprint 28F010 -> Libraries:28F010
Changed lines of the file:
@@
 $EndDescr
 $Comp
-L 28F010:28F010 U?
+L 28F010:28F010 U27
 U 1 1 61A2E775
 P 6100 1850
-F 0 "U?" H 7200 2237 60  0000 C CNN
+F 0 "U27" H 7200 2237 60  0000 C CNN
 F 1 "28F010" H 7200 2131 60  0000 C CNN
-F 2 "28F010" H 7200 2090 60  0001 C CNN
+F 2 "Libraries:28F010" H 7200 2090 60  0001 C CNN
 F 3 "" H 6100 1850 60  0000 C CNN
 	1    6100 1850
@@
 $EndComp
 $Comp
-L 28F010:28F010 U?
+L 28F010:28F010 U28
 U 1 1 61A3289A
 P 6100 4300
-F 0 "U?" H 7200 4687 60  0000 C CNN
+F 0 "U28" H 7200 4687 60  0000 C CNN
 F 1 "28F010" H 7200 4581 60  0000 C CNN
-F 2 "28F010" H 7200 4540 60  0001 C CNN
+F 2 "Libraries:28F010" H 7200 4540 60  0001 C CNN
 F 3 "" H 6100 4300 60  0000 C CNN
 	1    6100 4300
@@
 $EndComp
 $Comp
-L power:VCC #PWR?
+L power:VCC #PWR0198
 U 1 1 61A34CDA
 P 8300 4300
-F 0 "#PWR?" H 8300 4150 50  0001 C CNN
+F 0 "#PWR0198" H 8300 4150 50  0001 C CNN
 F 1 "VCC" H 8315 4473 50  0000 C CNN
 F 2 "" H 8300 4300 50  0001 C CNN
@@
 $EndComp
 $Comp
-L power:VCC #PWR?
+L power:VCC #PWR0199
 U 1 1 61A3D1A0
 P 8300 1850
-F 0 "#PWR?" H 8300 1700 50  0001 C CNN
+F 0 "#PWR0199" H 8300 1700 50  0001 C CNN
 F 1 "VCC" H 8315 2023 50  0000 C CNN
 F 2 "" H 8300 1850 50  0001 C CNN
@@
 $EndComp
 $Comp
-L power:VCC #PWR?
+L power:VCC #PWR0200
 U 1 1 61A3ED02
 P 3300 2500
-F 0 "#PWR?" H 3300 2350 50  0001 C CNN
+F 0 "#PWR0200" H 3300 2350 50  0001 C CNN
 F 1 "VCC" H 3315 2673 50  0000 C CNN
 F 2 "" H 3300 2500 50  0001 C CNN
@@
 $EndComp
 $Comp
-L power:GND #PWR?
+L power:GND #PWR0201
 U 1 1 61A3FEBA
 P 3000 3800
-F 0 "#PWR?" H 3000 3550 50  0001 C CNN
+F 0 "#PWR0201" H 3000 3550 50  0001 C CNN
 F 1 "GND" H 3005 3627 50  0000 C CNN
 F 2 "" H 3000 3800 50  0001 C CNN
@@
 $EndComp
 $Comp
-L power:GND #PWR?
+L power:GND #PWR0202
 U 1 1 61A413B4
 P 6100 3350
-F 0 "#PWR?" H 6100 3100 50  0001 C CNN
+F 0 "#PWR0202" H 6100 3100 50  0001 C CNN
 F 1 "GND" H 6105 3177 50  0000 C CNN
 F 2 "" H 6100 3350 50  0001 C CNN
@@
 NoConn ~ 8300 4500
 $Comp
-L power:GND #PWR?
+L power:GND #PWR0203
 U 1 1 61A44BE0
 P 6100 5800
-F 0 "#PWR?" H 6100 5550 50  0001 C CNN
+F 0 "#PWR0203" H 6100 5550 50  0001 C CNN
 F 1 "GND" H 6105 5627 50  0000 C CNN
 F 2 "" H 6100 5800 50  0001 C CNN
@@
 ~CE_HI_BYTE
 $Comp
-L power:+12V #PWR?
+L power:+12V #PWR0204
 U 1 1 61A56AD6
 P 6100 4300
-F 0 "#PWR?" H 6100 4150 50  0001 C CNN
+F 0 "#PWR0204" H 6100 4150 50  0001 C CNN
 F 1 "+12V" H 6115 4473 50  0000 C CNN
 F 2 "" H 6100 4300 50  0001 C CNN
@@
 $EndComp
 $Comp
-L power:+12V #PWR?
+L power:+12V #PWR0205
 U 1 1 61A5719E
 P 6100 1850
-F 0 "#PWR?" H 6100 1700 50  0001 C CNN
+F 0 "#PWR0205" H 6100 1700 50  0001 C CNN
 F 1 "+12V" H 6115 2023 50  0000 C CNN
 F 2 "" H 6100 1850 50  0001 C CNN
@@
 $EndComp
 $Comp
-L Device:C C?
+L Device:C C29
 U 1 1 61A5CD65
 P 900 6950
-F 0 "C?" H 1015 6996 50  0000 L CNN
+F 0 "C29" H 1015 6996 50  0000 L CNN
 F 1 "100nF" H 1015 6905 50  0000 L CNN
-F 2 "" H 938 6800 50  0001 C CNN
+F 2 "Capacitor_THT:C_Rect_L4.0mm_W2.5mm_P2.50mm" H 938 6800 50  0001 C CNN
 F 3 "~" H 900 6950 50  0001 C CNN
 	1    900  6950
@@
 $EndComp
 $Comp
-L Device:C C?
+L Device:C C30
 U 1 1 61A5F11A
 P 1400 6950
-F 0 "C?" H 1515 6996 50  0000 L CNN
+F 0 "C30" H 1515 6996 50  0000 L CNN
 F 1 "100nF" H 1515 6905 50  0000 L CNN
-F 2 "" H 1438 6800 50  0001 C CNN
+F 2 "Capacitor_THT:C_Rect_L4.0mm_W2.5mm_P2.50mm" H 1438 6800 50  0001 C CNN
 F 3 "~" H 1400 6950 50  0001 C CNN
 	1    1400 6950
@@
 $EndComp
 $Comp
-L Device:C C?
+L Device:C C31
 U 1 1 61A5F83C
 P 1850 6950
-F 0 "C?" H 1965 6996 50  0000 L CNN
+F 0 "C31" H 1965 6996 50  0000 L CNN
 F 1 "100nF" H 1965 6905 50  0000 L CNN
-F 2 "" H 1888 6800 50  0001 C CNN
+F 2 "Capacitor_THT:C_Rect_L4.0mm_W2.5mm_P2.50mm" H 1888 6800 50  0001 C CNN
 F 3 "~" H 1850 6950 50  0001 C CNN
 	1    1850 6950
@@
 $EndComp
 $Comp
-L Device:C C?
+L Device:C C32
 U 1 1 61A60007
 P 2300 6950
-F 0 "C?" H 2415 6996 50  0000 L CNN
+F 0 "C32" H 2415 6996 50  0000 L CNN
 F 1 "100nF" H 2415 6905 50  0000 L CNN
-F 2 "" H 2338 6800 50  0001 C CNN
+F 2 "Capacitor_THT:C_Rect_L4.0mm_W2.5mm_P2.50mm" H 2338 6800 50  0001 C CNN
 F 3 "~" H 2300 6950 50  0001 C CNN
 	1    2300 6950
@@
 	2300 7100 1850 7100
 $Comp
-L power:GND #PWR?
+L power:GND #PWR0206
 U 1 1 61A61AC2
 P 1850 7100
-F 0 "#PWR?" H 1850 6850 50  0001 C CNN
+F 0 "#PWR0206" H 1850 6850 50  0001 C CNN
 F 1 "GND" H 1855 6927 50  0000 C CNN
 F 2 "" H 1850 7100 50  0001 C CNN
@@
 	1400 6800 1150 6800
 $Comp
-L power:+12V #PWR?
+L power:+12V #PWR0207
 U 1 1 61A637CD
 P 1150 6800
-F 0 "#PWR?" H 1150 6650 50  0001 C CNN
+F 0 "#PWR0207" H 1150 6650 50  0001 C CNN
 F 1 "+12V" H 1165 6973 50  0000 C CNN
 F 2 "" H 1150 6800 50  0001 C CNN
@@
 	8400 1200 10800 1200
 $Comp
-L power:VCC #PWR?
+L power:VCC #PWR0208
 U 1 1 61AA5FAB
 P 2100 6800
-F 0 "#PWR?" H 2100 6650 50  0001 C CNN
+F 0 "#PWR0208" H 2100 6650 50  0001 C CNN
 F 1 "VCC" H 2115 6973 50  0000 C CNN
 F 2 "" H 2100 6800 50  0001 C CNN
@@
 ~CE_LOW_BYTE
 $Comp
-L 74xx:74LS138 U?
+L 74xx:74LS138 U25
 U 1 1 61B1DDB9
 P 3000 3100
-F 0 "U?" H 3000 3881 50  0000 C CNN
+F 0 "U25" H 3000 3881 50  0000 C CNN
 F 1 "74LS138" H 3000 3790 50  0000 C CNN
-F 2 "" H 3000 3100 50  0001 C CNN
+F 2 "Package_DIP:DIP-20_W7.62mm" H 3000 3100 50  0001 C CNN
 F 3 "http://www.ti.com/lit/gpn/sn74LS138" H 3000 3100 50  0001 C CNN
 	1    3000 3100
@@
 	3300 2500 3000 2500
 $Comp
-L power:VCC #PWR?
+L power:VCC #PWR0209
 U 1 1 61B31B97
 P 3300 4550
-F 0 "#PWR?" H 3300 4400 50  0001 C CNN
+F 0 "#PWR0209" H 3300 4400 50  0001 C CNN
 F 1 "VCC" H 3315 4723 50  0000 C CNN
 F 2 "" H 3300 4550 50  0001 C CNN
@@
 $EndComp
 $Comp
-L power:GND #PWR?
+L power:GND #PWR0210
 U 1 1 61B31B9D
 P 3000 5850
-F 0 "#PWR?" H 3000 5600 50  0001 C CNN
+F 0 "#PWR0210" H 3000 5600 50  0001 C CNN
 F 1 "GND" H 3005 5677 50  0000 C CNN
 F 2 "" H 3000 5850 50  0001 C CNN
@@
 $EndComp
 $Comp
-L 74xx:74LS138 U?
+L 74xx:74LS138 U26
 U 1 1 61B31BA3
 P 3000 5150
-F 0 "U?" H 3000 5931 50  0000 C CNN
+F 0 "U26" H 3000 5931 50  0000 C CNN
 F 1 "74LS138" H 3000 5840 50  0000 C CNN
-F 2 "" H 3000 5150 50  0001 C CNN
+F 2 "Package_DIP:DIP-20_W7.62mm" H 3000 5150 50  0001 C CNN
 F 3 "http://www.ti.com/lit/gpn/sn74LS138" H 3000 5150 50  0001 C CNN
 	1    3000 5150
@@
 	2200 3000 2200 3500
 $Comp
-L power:GND #PWR?
+L power:GND #PWR0211
 U 1 1 61BA2F85
 P 2200 5550
-F 0 "#PWR?" H 2200 5300 50  0001 C CNN
+F 0 "#PWR0211" H 2200 5300 50  0001 C CNN
 F 1 "GND" H 2205 5377 50  0000 C CNN
 F 2 "" H 2200 5550 50  0001 C CNN
@@
 	1850 2800 2500 2800
 $Comp
-L Device:C C?
+L Device:C C33
 U 1 1 61C77471
 P 2750 6950
-F 0 "C?" H 2865 6996 50  0000 L CNN
+F 0 "C33" H 2865 6996 50  0000 L CNN
 F 1 "100nF" H 2865 6905 50  0000 L CNN
-F 2 "" H 2788 6800 50  0001 C CNN
+F 2 "Capacitor_THT:C_Rect_L4.0mm_W2.5mm_P2.50mm" H 2788 6800 50  0001 C CNN
 F 3 "~" H 2750 6950 50  0001 C CNN
 	1    2750 6950
@@
 $EndComp
 $Comp
-L Device:C C?
+L Device:C C34
 U 1 1 61C7789A
 P 3200 6950
-F 0 "C?" H 3315 6996 50  0000 L CNN
+F 0 "C34" H 3315 6996 50  0000 L CNN
 F 1 "100nF" H 3315 6905 50  0000 L CNN
-F 2 "" H 3238 6800 50  0001 C CNN
+F 2 "Capacitor_THT:C_Rect_L4.0mm_W2.5mm_P2.50mm" H 3238 6800 50  0001 C CNN
 F 3 "~" H 3200 6950 50  0001 C CNN
 	1    3200 6950

Commit message: Route some more, starting re-doing memory routing
Parts:
- U25, U26: footprint Package_DIP:DIP-20_W7.62mm -> Package_DIP:DIP-16_W7.62mm
Changed lines of the file:
@@
 F 0 "U25" H 3000 3881 50  0000 C CNN
 F 1 "74LS138" H 3000 3790 50  0000 C CNN
-F 2 "Package_DIP:DIP-20_W7.62mm" H 3000 3100 50  0001 C CNN
+F 2 "Package_DIP:DIP-16_W7.62mm" H 3000 3100 50  0001 C CNN
 F 3 "http://www.ti.com/lit/gpn/sn74LS138" H 3000 3100 50  0001 C CNN
 	1    3000 3100
@@
 F 0 "U26" H 3000 5931 50  0000 C CNN
 F 1 "74LS138" H 3000 5840 50  0000 C CNN
-F 2 "Package_DIP:DIP-20_W7.62mm" H 3000 5150 50  0001 C CNN
+F 2 "Package_DIP:DIP-16_W7.62mm" H 3000 5150 50  0001 C CNN
 F 3 "http://www.ti.com/lit/gpn/sn74LS138" H 3000 5150 50  0001 C CNN
 	1    3000 5150
