File: UART-interface.sch (KiCad schematic (older format))
At the start: 19 parts

Commit message: Replaced MWTC MRDC IOWC IORC with WR RD; buffered control bus; consolidated logic gates
Parts:
- removed U? (x4): 74LS02, symbol 74xx:74LS02
- removed U? (x5): 74LS00, symbol 74xx:74LS00
- removed U? (x5): 74LS08, symbol 74xx:74LS08
- added R?: 1k, symbol Device:R
Connections:
- net labels added: ~CS, ~RD, ~WR
- net labels removed: A10, A11, A12, A13, A14, A15, A4, A5, A6, A7, A8, A9, AE, M\~IO, ~BHE, ~IORC, ~IOWC
- wire segments 122 -> 86
Other:
- note removed: "Address Decoding\n0x1111_1111_1110_xxx1"
