File: UART-interface.sch (KiCad schematic (older format))
At the start: 6 parts

Commit message: General edits; removed floating inputs
Connections:
- net GND: now also U?.16 (T4IN), U?.22 (T5IN)
- no-connect marks 10 -> 8
Changed lines of the file:
@@
 $Descr A4 11693 8268
 encoding utf-8
-Sheet 5 15
+Sheet 4 15
 Title "UART-interface"
 Date ""
@@
 	8900 4750 8850 4750
 Wire Wire Line
-	8900 4750 8900 5650
+	8900 4750 8900 5150
 Connection ~ 8900 4750
 Wire Wire Line
@@
 	9200 5350 9200 1300
 NoConn ~ 6250 4350
-NoConn ~ 8850 4550
 NoConn ~ 8850 4850
-NoConn ~ 8850 5150
 NoConn ~ 3450 1900
 NoConn ~ 3450 2200
@@
 Wire Notes Line
 	3650 4450 600  4450
+Wire Wire Line
+	8850 4550 8900 4550
+Wire Wire Line
+	8900 4550 8900 4650
+Connection ~ 8900 4650
+Wire Wire Line
+	8850 5150 8900 5150
 Wire Bus Line
 	1250 1800 1250 2100
 Wire Bus Line
 	1250 900  1250 1700
+Connection ~ 8900 5150
+Wire Wire Line
+	8900 5150 8900 5650
 $EndSCHEMATC

Commit message: Updates to pass ERC
Changed lines of the file:
@@
 D15
 Text HLabel 1250 900  0    50   BiDi ~ 0
-DATA_BUS
+D[0..15]
 Text Notes 10800 850  2    50   ~ 0
 UART Interface\n I/O  Addresses 0xFFEF to 0xFFE1
@@
 U 1 1 61A48DF3
 P 9850 3000
+AR Path="/61A48DF3" Ref="J?"  Part="1"
+AR Path="/61A42887/61A48DF3" Ref="J?"  Part="1"
 F 0 "J?" H 10678 2653 60  0000 L CNN
 F 1 "DSUB-9" H 10678 2547 60  0000 L CNN
@@
 	1450 2000 1350 2000
 Text HLabel 1250 1800 0    50   Input ~ 0
-ADDRESS_BUS
+A[0..19]
 Text Label 1350 2000 0    50   ~ 0
 A1
@@
 Wire Wire Line
 	8850 5150 8900 5150
+Connection ~ 8900 5150
+Wire Wire Line
+	8900 5150 8900 5650
 Wire Bus Line
 	1250 1800 1250 2100
 Wire Bus Line
 	1250 900  1250 1700
-Connection ~ 8900 5150
-Wire Wire Line
-	8900 5150 8900 5650
 $EndSCHEMATC

Commit message: Assign footprints for most symbols
Parts:
- C5, C6: renamed from C?; footprint (none) -> Capacitor_THT:C_Rect_L4.0mm_W2.5mm_P2.50mm
- J6: renamed from J?; footprint DSUB-9 -> Libraries:DSUB-9
- R3: renamed from R?; footprint (none) -> Resistor_THT:R_Axial_DIN0207_L6.3mm_D2.5mm_P10.16mm_Horizontal
- U3: renamed from U?; footprint max235cpg -> Libraries:max235cpg
- gave numbers to parts that had none: 1
Changed lines of the file:
@@
 $EndDescr
 $Comp
-L power:VCC #PWR?
+L power:VCC #PWR0109
 U 1 1 61A42AAB
 P 9850 1550
-F 0 "#PWR?" H 9850 1400 50  0001 C CNN
+F 0 "#PWR0109" H 9850 1400 50  0001 C CNN
 F 1 "VCC" H 9865 1723 50  0000 C CNN
 F 2 "" H 9850 1550 50  0001 C CNN
@@
 $EndComp
 $Comp
-L power:GND #PWR?
+L power:GND #PWR0110
 U 1 1 61A4364E
 P 9850 1850
-F 0 "#PWR?" H 9850 1600 50  0001 C CNN
+F 0 "#PWR0110" H 9850 1600 50  0001 C CNN
 F 1 "GND" H 9855 1677 50  0000 C CNN
 F 2 "" H 9850 1850 50  0001 C CNN
@@
 $EndComp
 $Comp
-L Device:C C?
+L Device:C C5
 U 1 1 61A43B7F
 P 9850 1700
-F 0 "C?" H 9965 1746 50  0000 L CNN
+F 0 "C5" H 9965 1746 50  0000 L CNN
 F 1 "100nF" H 9965 1655 50  0000 L CNN
-F 2 "" H 9888 1550 50  0001 C CNN
+F 2 "Capacitor_THT:C_Rect_L4.0mm_W2.5mm_P2.50mm" H 9888 1550 50  0001 C CNN
 F 3 "~" H 9850 1700 50  0001 C CNN
 	1    9850 1700
@@
 $EndComp
 $Comp
-L Interface_UART:16550 U?
+L Interface_UART:16550 U2
 U 1 1 61A498A6
 P 2450 2500
-F 0 "U?" H 2450 4381 50  0000 C CNN
+F 0 "U2" H 2450 4381 50  0000 C CNN
 F 1 "16550" H 2450 4290 50  0000 C CNN
 F 2 "Package_DIP:DIP-40_W15.24mm" H 2450 2500 50  0001 C CIN
@@
 $EndComp
 $Comp
-L Device:C C?
+L Device:C C6
 U 1 1 61A4B29D
 P 10350 1700
-F 0 "C?" H 10465 1746 50  0000 L CNN
+F 0 "C6" H 10465 1746 50  0000 L CNN
 F 1 "100nF" H 10465 1655 50  0000 L CNN
-F 2 "" H 10388 1550 50  0001 C CNN
+F 2 "Capacitor_THT:C_Rect_L4.0mm_W2.5mm_P2.50mm" H 10388 1550 50  0001 C CNN
 F 3 "~" H 10350 1700 50  0001 C CNN
 	1    10350 1700
@@
 Connection ~ 9850 1850
 $Comp
-L power:VCC #PWR?
+L power:VCC #PWR0111
 U 1 1 61A4DA12
 P 2700 800
-F 0 "#PWR?" H 2700 650 50  0001 C CNN
+F 0 "#PWR0111" H 2700 650 50  0001 C CNN
 F 1 "VCC" H 2715 973 50  0000 C CNN
 F 2 "" H 2700 800 50  0001 C CNN
@@
 	1000 3500 1000 3700
 $Comp
-L power:GND #PWR?
+L power:GND #PWR0112
 U 1 1 61A503DE
 P 2450 4200
-F 0 "#PWR?" H 2450 3950 50  0001 C CNN
+F 0 "#PWR0112" H 2450 3950 50  0001 C CNN
 F 1 "GND" H 2455 4027 50  0000 C CNN
 F 2 "" H 2450 4200 50  0001 C CNN
@@
 $EndComp
 $Comp
-L power:GND #PWR?
+L power:GND #PWR0113
 U 1 1 61A64B26
 P 1000 4050
-F 0 "#PWR?" H 1000 3800 50  0001 C CNN
+F 0 "#PWR0113" H 1000 3800 50  0001 C CNN
 F 1 "GND" H 1005 3877 50  0000 C CNN
 F 2 "" H 1000 4050 50  0001 C CNN
@@
 	3550 3900 3450 3900
 $Comp
-L power:VCC #PWR?
+L power:VCC #PWR0114
 U 1 1 61AAB957
 P 6200 4150
-F 0 "#PWR?" H 6200 4000 50  0001 C CNN
+F 0 "#PWR0114" H 6200 4000 50  0001 C CNN
 F 1 "VCC" H 6215 4323 50  0000 C CNN
 F 2 "" H 6200 4150 50  0001 C CNN
@@
 $EndComp
 $Comp
-L power:GND #PWR?
+L power:GND #PWR0115
 U 1 1 61A86B8C
 P 8900 5650
-F 0 "#PWR?" H 8900 5400 50  0001 C CNN
+F 0 "#PWR0115" H 8900 5400 50  0001 C CNN
 F 1 "GND" H 8905 5477 50  0000 C CNN
 F 2 "" H 8900 5650 50  0001 C CNN
@@
 P 9850 3000
 AR Path="/61A48DF3" Ref="J?"  Part="1"
-AR Path="/61A42887/61A48DF3" Ref="J?"  Part="1"
-F 0 "J?" H 10678 2653 60  0000 L CNN
+AR Path="/61A42887/61A48DF3" Ref="J6"  Part="1"
+F 0 "J6" H 10678 2653 60  0000 L CNN
 F 1 "DSUB-9" H 10678 2547 60  0000 L CNN
-F 2 "DSUB-9" H 10450 2640 60  0001 C CNN
+F 2 "Libraries:DSUB-9" H 10450 2640 60  0001 C CNN
 F 3 "" H 9850 3000 60  0000 C CNN
 	1    9850 3000
@@
 $EndComp
 $Comp
-L max235cpg:max235cpg U?
+L max235cpg:max235cpg U3
 U 1 1 61B898E2
 P 6250 4350
-F 0 "U?" H 7550 4737 60  0000 C CNN
+F 0 "U3" H 7550 4737 60  0000 C CNN
 F 1 "max235cpg" H 7550 4631 60  0000 C CNN
-F 2 "max235cpg" H 7550 4590 60  0001 C CNN
+F 2 "Libraries:max235cpg" H 7550 4590 60  0001 C CNN
 F 3 "" H 6250 4350 60  0000 C CNN
 	1    6250 4350
@@
 	9850 3800 9150 3800
 $Comp
-L power:GND #PWR?
+L power:GND #PWR0116
 U 1 1 624418EE
 P 6150 5650
-F 0 "#PWR?" H 6150 5400 50  0001 C CNN
+F 0 "#PWR0116" H 6150 5400 50  0001 C CNN
 F 1 "GND" H 6155 5477 50  0000 C CNN
 F 2 "" H 6150 5650 50  0001 C CNN
@@
 	9750 3400 9750 3900
 $Comp
-L power:GND #PWR?
+L power:GND #PWR0117
 U 1 1 624E8BB9
 P 9750 3900
-F 0 "#PWR?" H 9750 3650 50  0001 C CNN
+F 0 "#PWR0117" H 9750 3650 50  0001 C CNN
 F 1 "GND" H 9755 3727 50  0000 C CNN
 F 2 "" H 9750 3900 50  0001 C CNN
@@
 	1000 3700 1000 4050
 $Comp
-L Device:R R?
+L Device:R R3
 U 1 1 61C6139A
 P 1050 2300
-F 0 "R?" V 1257 2300 50  0000 C CNN
+F 0 "R3" V 1257 2300 50  0000 C CNN
 F 1 "1k" V 1166 2300 50  0000 C CNN
-F 2 "" V 980 2300 50  0001 C CNN
+F 2 "Resistor_THT:R_Axial_DIN0207_L6.3mm_D2.5mm_P10.16mm_Horizontal" V 980 2300 50  0001 C CNN
 F 3 "~" H 1050 2300 50  0001 C CNN
 	1    1050 2300
@@
 $EndComp
 $Comp
-L power:VCC #PWR?
+L power:VCC #PWR0118
 U 1 1 61C62224
 P 800 2300
-F 0 "#PWR?" H 800 2150 50  0001 C CNN
+F 0 "#PWR0118" H 800 2150 50  0001 C CNN
 F 1 "VCC" H 815 2473 50  0000 C CNN
 F 2 "" H 800 2300 50  0001 C CNN
