File: external-connectors.sch (KiCad schematic (older format))
At the start: 7 parts

Commit message: Replaced MWTC MRDC IOWC IORC with WR RD; buffered control bus; consolidated logic gates
Connections:
- net ~MWTC is gone; now on net RESET: J?.5 (Pin_5)
- net RESET: no longer J?.7 (Pin_7)
- net ~RD: now reaches J?.8 (Pin_8)
- net ~IORC renamed M\~IO
- net ~IOWC renamed ~WR
- net ~MRDC renamed PCLK
Changed lines of the file:
@@
 $Descr A4 11693 8268
 encoding utf-8
-Sheet 3 10
+Sheet 2 11
 Title "external-connectors"
 Date ""
@@
 Wire Wire Line
 	8200 3600 7500 3600
-Text HLabel 4100 4750 0    50   Output ~ 0
+Text HLabel 4100 4750 0    50   Input ~ 0
 CLK
-Text HLabel 4100 4850 0    50   UnSpc ~ 0
-~MRDC
-Text HLabel 4100 4950 0    50   Input ~ 0
-~MWTC
-Text HLabel 4600 4850 2    50   Output ~ 0
-~IORC
-Text HLabel 4600 4950 2    50   Output ~ 0
-~IOWC
+Text HLabel 4100 4850 0    50   Input ~ 0
+PCLK
 $Comp
 L Connector_Generic:Conn_02x08_Odd_Even J?
@@
 	1    0    0    -1
 $EndComp
-Text HLabel 4100 5050 0    50   Input ~ 0
+Text HLabel 4100 4950 0    50   Input ~ 0
 RESET
-Text HLabel 4600 4750 2    50   Output ~ 0
+Text HLabel 4600 4750 2    50   Input ~ 0
 ~BHE
 $Comp
@@
 Wire Bus Line
 	1900 1950 4650 1950
+Text HLabel 4600 4850 2    50   Input ~ 0
+M\~IO
+Text HLabel 4600 4950 2    50   Input ~ 0
+~WR
+Text HLabel 4600 5050 2    50   Input ~ 0
+~RD
 $EndSCHEMATC
