File: peripheral-interface.sch (KiCad schematic (older format))
At the start: 5 parts

Commit message: Updates to pass ERC
Changed lines of the file:
@@
 $EndComp
 Text HLabel 4050 3000 0    50   Input ~ 0
-ADDRESS_BUS
+A[0..19]
 Entry Wire Line
 	4050 3175 4150 3275
@@
 $EndComp
 Text HLabel 4050 4500 0    50   BiDi ~ 0
-DATA_BUS
+D[0..15]
 Entry Wire Line
 	4050 4375 4150 4275
