File: interrupt-controller.sch (KiCad schematic (older format))
At the start: 14 parts, among them J16 IR4-IR7, SW2 SW_Push, U13 8259, U14 74LS14

Commit message: begin pcb layout
Parts:
- J16: footprint Connector_PinHeader_2.54mm:PinHeader_1x03_P2.54mm_Vertical -> Connector_PinHeader_2.54mm:PinHeader_1x04_P2.54mm_Vertical
- SW2: value SW_Push -> IR0
Changed lines of the file:
@@
 F 0 "J16" H 5580 2242 50  0000 L CNN
 F 1 "IR4-IR7" H 5580 2151 50  0000 L CNN
-F 2 "Connector_PinHeader_2.54mm:PinHeader_1x03_P2.54mm_Vertical" H 5500 2250 50  0001 C CNN
+F 2 "Connector_PinHeader_2.54mm:PinHeader_1x04_P2.54mm_Vertical" H 5500 2250 50  0001 C CNN
 F 3 "~" H 5500 2250 50  0001 C CNN
 	1    5500 2250
@@
 P 2450 6200
 F 0 "SW2" H 2450 6485 50  0000 C CNN
-F 1 "SW_Push" H 2450 6394 50  0000 C CNN
+F 1 "IR0" H 2450 6394 50  0000 C CNN
 F 2 "Button_Switch_Keyboard:SW_Cherry_MX_1.00u_PCB" H 2450 6400 50  0001 C CNN
 F 3 "~" H 2450 6400 50  0001 C CNN
