File: peripheral-interface-odd.sch (KiCad schematic (older format))
At the start: 5 parts

Commit message: Fix wiring in root sheet
Parts:
- removed C?: 100nF, symbol Device:C
- removed J? (x2): Conn_01x08, symbol Connector_Generic:Conn_01x08
- removed U?: 8255, Package_DIP:DIP-40_W15.24mm, symbol Interface:8255
- added C?: 100nF, symbol Device:C
- added J? (x2): Conn_01x08, symbol Connector_Generic:Conn_01x08
- added U?: 8255, Package_DIP:DIP-40_W15.24mm, symbol Interface:8255
Connections:
- net A1: now also U?.8 (A1)
- net A2: now also U?.9 (A0)
- net D10: now also U?.32 (D2)
- net D11: now also U?.31 (D3)
- net D12: now also U?.30 (D4)
- net D13: now also U?.29 (D5)
- net D14: now also U?.28 (D6)
- net D15: now also U?.27 (D7)
- net D8: now also U?.34 (D0)
- net D9: now also U?.33 (D1)
- net GND: now also C?.2, U?.7 (GND)
- net RESET: now also U?.35 (RESET)
- net VCC: now also C?.1, U?.26 (VCC)
- net ~CS: now also U?.6 (~CS~)
- net ~RD: now also U?.5 (~RD~)
- net ~WR: now also U?.36 (~WR~)
- net at J?.1 (Pin_1): now also U?.18 (PB0)
- net at J?.2 (Pin_2): now also U?.19 (PB1)
- net at J?.3 (Pin_3): now also U?.20 (PB2)
- net at J?.4 (Pin_4): now also U?.21 (PB3)
- net at J?.5 (Pin_5): now also U?.22 (PB4)
- net at J?.6 (Pin_6): now also U?.23 (PB5)
- net at J?.7 (Pin_7): now also U?.24 (PB6)
- net at J?.8 (Pin_8): now also U?.25 (PB7)
- new net: J?.4 (Pin_4), U?.1 (PA3)
- new net: J?.8 (Pin_8), U?.10 (PC7)
- new net: J?.7 (Pin_7), U?.11 (PC6)
- new net: J?.6 (Pin_6), U?.12 (PC5)
- new net: J?.5 (Pin_5), U?.13 (PC4)
- new net: J?.1 (Pin_1), U?.14 (PC0)
- new net: J?.2 (Pin_2), U?.15 (PC1)
- new net: J?.3 (Pin_3), U?.16 (PC2)
- new net: J?.4 (Pin_4), U?.17 (PC3)
- new net: J?.3 (Pin_3), U?.2 (PA2)
- new net: J?.2 (Pin_2), U?.3 (PA1)
- new net: J?.8 (Pin_8), U?.37 (PA7)
- new net: J?.7 (Pin_7), U?.38 (PA6)
- new net: J?.6 (Pin_6), U?.39 (PA5)
- new net: J?.1 (Pin_1), U?.4 (PA0)
- new net: J?.5 (Pin_5), U?.40 (PA4)
Changed lines of the file:
@@
 $Descr A4 11693 8268
 encoding utf-8
-Sheet 8 14
+Sheet 8 15
 Title "Peripheral Interface"
 Date ""
@@
 $Comp
 L Connector_Generic:Conn_01x08 J?
-U 1 1 61C3F083
+U 1 1 61ABA7C3
 P 5900 4475
-AR Path="/61BFC8AC/61C0115A/61C3F083" Ref="J?"  Part="1"
-AR Path="/61BFC8AC/61C2038B/61C3F083" Ref="J?"  Part="1"
-AR Path="/61BFC8AC/61C20895/61C3F083" Ref="J?"  Part="1"
-AR Path="/61C40B21/61C3F083" Ref="J?"  Part="1"
-AR Path="/61C417C6/61C3F083" Ref="J?"  Part="1"
-AR Path="/61C41B68/61C3F083" Ref="J?"  Part="1"
+AR Path="/61BFC8AC/61C0115A/61ABA7C3" Ref="J?"  Part="1"
+AR Path="/61BFC8AC/61C2038B/61ABA7C3" Ref="J?"  Part="1"
+AR Path="/61BFC8AC/61C20895/61ABA7C3" Ref="J?"  Part="1"
+AR Path="/61C40B21/61ABA7C3" Ref="J?"  Part="1"
+AR Path="/61C417C6/61ABA7C3" Ref="J?"  Part="1"
+AR Path="/61C41B68/61ABA7C3" Ref="J?"  Part="1"
 F 0 "J?" H 5980 4467 50  0000 L CNN
 F 1 "Conn_01x08" H 5980 4376 50  0000 L CNN
@@
 $Comp
 L Connector_Generic:Conn_01x08 J?
-U 1 1 61C397EF
+U 1 1 61ABA7C1
 P 5900 2675
-AR Path="/61BFC8AC/61C0115A/61C397EF" Ref="J?"  Part="1"
-AR Path="/61BFC8AC/61C2038B/61C397EF" Ref="J?"  Part="1"
-AR Path="/61BFC8AC/61C20895/61C397EF" Ref="J?"  Part="1"
-AR Path="/61C40B21/61C397EF" Ref="J?"  Part="1"
-AR Path="/61C417C6/61C397EF" Ref="J?"  Part="1"
-AR Path="/61C41B68/61C397EF" Ref="J?"  Part="1"
+AR Path="/61BFC8AC/61C0115A/61ABA7C1" Ref="J?"  Part="1"
+AR Path="/61BFC8AC/61C2038B/61ABA7C1" Ref="J?"  Part="1"
+AR Path="/61BFC8AC/61C20895/61ABA7C1" Ref="J?"  Part="1"
+AR Path="/61C40B21/61ABA7C1" Ref="J?"  Part="1"
+AR Path="/61C417C6/61ABA7C1" Ref="J?"  Part="1"
+AR Path="/61C41B68/61ABA7C1" Ref="J?"  Part="1"
 F 0 "J?" H 5980 2667 50  0000 L CNN
 F 1 "Conn_01x08" H 5980 2576 50  0000 L CNN
@@
 $Comp
 L power:GND #PWR?
-U 1 1 61C2D896
+U 1 1 61ABA7C0
 P 5000 5275
-AR Path="/61BFC8AC/61C0115A/61C2D896" Ref="#PWR?"  Part="1"
-AR Path="/61BFC8AC/61C2038B/61C2D896" Ref="#PWR?"  Part="1"
-AR Path="/61BFC8AC/61C20895/61C2D896" Ref="#PWR?"  Part="1"
-AR Path="/61C40B21/61C2D896" Ref="#PWR?"  Part="1"
-AR Path="/61C417C6/61C2D896" Ref="#PWR?"  Part="1"
-AR Path="/61C41B68/61C2D896" Ref="#PWR?"  Part="1"
+AR Path="/61BFC8AC/61C0115A/61ABA7C0" Ref="#PWR?"  Part="1"
+AR Path="/61BFC8AC/61C2038B/61ABA7C0" Ref="#PWR?"  Part="1"
+AR Path="/61BFC8AC/61C20895/61ABA7C0" Ref="#PWR?"  Part="1"
+AR Path="/61C40B21/61ABA7C0" Ref="#PWR?"  Part="1"
+AR Path="/61C417C6/61ABA7C0" Ref="#PWR?"  Part="1"
+AR Path="/61C41B68/61ABA7C0" Ref="#PWR?"  Part="1"
 F 0 "#PWR?" H 5000 5025 50  0001 C CNN
 F 1 "GND" H 5005 5102 50  0000 C CNN
@@
 $Comp
 L power:VCC #PWR?
-U 1 1 61C2CF0A
+U 1 1 61ABA7BF
 P 5000 2075
-AR Path="/61BFC8AC/61C0115A/61C2CF0A" Ref="#PWR?"  Part="1"
-AR Path="/61BFC8AC/61C2038B/61C2CF0A" Ref="#PWR?"  Part="1"
-AR Path="/61BFC8AC/61C20895/61C2CF0A" Ref="#PWR?"  Part="1"
-AR Path="/61C40B21/61C2CF0A" Ref="#PWR?"  Part="1"
-AR Path="/61C417C6/61C2CF0A" Ref="#PWR?"  Part="1"
-AR Path="/61C41B68/61C2CF0A" Ref="#PWR?"  Part="1"
+AR Path="/61BFC8AC/61C0115A/61ABA7BF" Ref="#PWR?"  Part="1"
+AR Path="/61BFC8AC/61C2038B/61ABA7BF" Ref="#PWR?"  Part="1"
+AR Path="/61BFC8AC/61C20895/61ABA7BF" Ref="#PWR?"  Part="1"
+AR Path="/61C40B21/61ABA7BF" Ref="#PWR?"  Part="1"
+AR Path="/61C417C6/61ABA7BF" Ref="#PWR?"  Part="1"
+AR Path="/61C41B68/61ABA7BF" Ref="#PWR?"  Part="1"
 F 0 "#PWR?" H 5000 1925 50  0001 C CNN
 F 1 "VCC" H 5015 2248 50  0000 C CNN
@@
 $Comp
 L Interface:8255 U?
-U 1 1 61C013ED
+U 1 1 61ABA7BE
 P 5000 3675
-AR Path="/61BFC8AC/61C0115A/61C013ED" Ref="U?"  Part="1"
-AR Path="/61BFC8AC/61C2038B/61C013ED" Ref="U?"  Part="1"
-AR Path="/61BFC8AC/61C20895/61C013ED" Ref="U?"  Part="1"
-AR Path="/61BFC8AC/61C20AD2/61C013ED" Ref="U?"  Part="1"
-AR Path="/61BFC8AC/61C20ADE/61C013ED" Ref="U?"  Part="1"
-AR Path="/61BFC8AC/61C20AEA/61C013ED" Ref="U?"  Part="1"
-AR Path="/61C40B21/61C013ED" Ref="U?"  Part="1"
-AR Path="/61C417C6/61C013ED" Ref="U?"  Part="1"
-AR Path="/61C41B68/61C013ED" Ref="U?"  Part="1"
+AR Path="/61BFC8AC/61C0115A/61ABA7BE" Ref="U?"  Part="1"
+AR Path="/61BFC8AC/61C2038B/61ABA7BE" Ref="U?"  Part="1"
+AR Path="/61BFC8AC/61C20895/61ABA7BE" Ref="U?"  Part="1"
+AR Path="/61BFC8AC/61C20AD2/61ABA7BE" Ref="U?"  Part="1"
+AR Path="/61BFC8AC/61C20ADE/61ABA7BE" Ref="U?"  Part="1"
+AR Path="/61BFC8AC/61C20AEA/61ABA7BE" Ref="U?"  Part="1"
+AR Path="/61C40B21/61ABA7BE" Ref="U?"  Part="1"
+AR Path="/61C417C6/61ABA7BE" Ref="U?"  Part="1"
+AR Path="/61C41B68/61ABA7BE" Ref="U?"  Part="1"
 F 0 "U?" H 5000 3775 50  0000 C CNN
 F 1 "8255" H 5000 3675 50  0000 C CNN
@@
 $Comp
 L Device:C C?
-U 1 1 61C5D8E9
+U 1 1 61ABA7C4
 P 7875 3375
-AR Path="/61C417C6/61C5D8E9" Ref="C?"  Part="1"
-AR Path="/61C41B68/61C5D8E9" Ref="C?"  Part="1"
-AR Path="/61C40B21/61C5D8E9" Ref="C?"  Part="1"
+AR Path="/61C417C6/61ABA7C4" Ref="C?"  Part="1"
+AR Path="/61C41B68/61ABA7C4" Ref="C?"  Part="1"
+AR Path="/61C40B21/61ABA7C4" Ref="C?"  Part="1"
 F 0 "C?" H 7990 3421 50  0000 L CNN
 F 1 "100nF" H 7990 3330 50  0000 L CNN
@@
 $Comp
 L power:VCC #PWR?
-U 1 1 61C60AFC
+U 1 1 61ABA7C5
 P 7875 3225
-AR Path="/61C417C6/61C60AFC" Ref="#PWR?"  Part="1"
-AR Path="/61C41B68/61C60AFC" Ref="#PWR?"  Part="1"
-AR Path="/61C40B21/61C60AFC" Ref="#PWR?"  Part="1"
+AR Path="/61C417C6/61ABA7C5" Ref="#PWR?"  Part="1"
+AR Path="/61C41B68/61ABA7C5" Ref="#PWR?"  Part="1"
+AR Path="/61C40B21/61ABA7C5" Ref="#PWR?"  Part="1"
 F 0 "#PWR?" H 7875 3075 50  0001 C CNN
 F 1 "VCC" H 7890 3398 50  0000 C CNN

Commit message: General edits; removed floating inputs
Connections:
- net A1: now also U?.9 (A0); no longer U?.8 (A1)
- net A2: now also U?.8 (A1); no longer U?.9 (A0)
Changed lines of the file:
@@
 $Descr A4 11693 8268
 encoding utf-8
-Sheet 8 15
+Sheet 7 15
 Title "Peripheral Interface"
 Date ""
@@
 	4050 3075 4150 3175
 Text Label 4150 3275 0    50   ~ 0
-A1
-Text Label 4150 3175 0    50   ~ 0
 A2
 Wire Wire Line
@@
 Wire Bus Line
 	4050 3675 4050 4500
+Text Label 4150 3175 0    50   ~ 0
+A1
 $EndSCHEMATC

Commit message: Updates to pass ERC
Changed lines of the file:
@@
 $EndComp
 Text HLabel 4050 3000 0    50   Input ~ 0
-ADDRESS_BUS
+A[0..19]
 Entry Wire Line
 	4050 3175 4150 3275
@@
 $EndComp
 Text HLabel 4050 4500 0    50   BiDi ~ 0
-DATA_BUS
+D[0..15]
 Entry Wire Line
 	4050 4375 4150 4275

Commit message: Assign footprints for most symbols
Parts:
- C13: renamed from C?; footprint (none) -> Capacitor_THT:C_Rect_L4.0mm_W2.5mm_P2.50mm
- J10, J11, J12: renamed from J?; footprint (none) -> Connector_PinHeader_2.54mm:PinHeader_1x08_P2.54mm_Vertical
- gave numbers to parts that had none: 1
Changed lines of the file:
@@
 $Descr A4 11693 8268
 encoding utf-8
-Sheet 7 15
+Sheet 6 15
 Title "Peripheral Interface"
 Date ""
@@
 AR Path="/61BFC8AC/61C2038B/61ABA7C3" Ref="J?"  Part="1"
 AR Path="/61BFC8AC/61C20895/61ABA7C3" Ref="J?"  Part="1"
-AR Path="/61C40B21/61ABA7C3" Ref="J?"  Part="1"
+AR Path="/61C40B21/61ABA7C3" Ref="J12"  Part="1"
 AR Path="/61C417C6/61ABA7C3" Ref="J?"  Part="1"
-AR Path="/61C41B68/61ABA7C3" Ref="J?"  Part="1"
-F 0 "J?" H 5980 4467 50  0000 L CNN
+AR Path="/61C41B68/61ABA7C3" Ref="J9"  Part="1"
+F 0 "J9" H 5980 4467 50  0000 L CNN
 F 1 "Conn_01x08" H 5980 4376 50  0000 L CNN
-F 2 "" H 5900 4475 50  0001 C CNN
+F 2 "Connector_PinHeader_2.54mm:PinHeader_1x08_P2.54mm_Vertical" H 5900 4475 50  0001 C CNN
 F 3 "~" H 5900 4475 50  0001 C CNN
 	1    5900 4475
@@
 AR Path="/61BFC8AC/61C2038B/61C3EA07" Ref="J?"  Part="1"
 AR Path="/61BFC8AC/61C20895/61C3EA07" Ref="J?"  Part="1"
-AR Path="/61C40B21/61C3EA07" Ref="J?"  Part="1"
+AR Path="/61C40B21/61C3EA07" Ref="J11"  Part="1"
 AR Path="/61C417C6/61C3EA07" Ref="J?"  Part="1"
-AR Path="/61C41B68/61C3EA07" Ref="J?"  Part="1"
-F 0 "J?" H 5980 3567 50  0000 L CNN
+AR Path="/61C41B68/61C3EA07" Ref="J8"  Part="1"
+F 0 "J8" H 5980 3567 50  0000 L CNN
 F 1 "Conn_01x08" H 5980 3476 50  0000 L CNN
-F 2 "" H 5900 3575 50  0001 C CNN
+F 2 "Connector_PinHeader_2.54mm:PinHeader_1x08_P2.54mm_Vertical" H 5900 3575 50  0001 C CNN
 F 3 "~" H 5900 3575 50  0001 C CNN
 	1    5900 3575
@@
 AR Path="/61BFC8AC/61C2038B/61ABA7C1" Ref="J?"  Part="1"
 AR Path="/61BFC8AC/61C20895/61ABA7C1" Ref="J?"  Part="1"
-AR Path="/61C40B21/61ABA7C1" Ref="J?"  Part="1"
+AR Path="/61C40B21/61ABA7C1" Ref="J10"  Part="1"
 AR Path="/61C417C6/61ABA7C1" Ref="J?"  Part="1"
-AR Path="/61C41B68/61ABA7C1" Ref="J?"  Part="1"
-F 0 "J?" H 5980 2667 50  0000 L CNN
+AR Path="/61C41B68/61ABA7C1" Ref="J7"  Part="1"
+F 0 "J7" H 5980 2667 50  0000 L CNN
 F 1 "Conn_01x08" H 5980 2576 50  0000 L CNN
-F 2 "" H 5900 2675 50  0001 C CNN
+F 2 "Connector_PinHeader_2.54mm:PinHeader_1x08_P2.54mm_Vertical" H 5900 2675 50  0001 C CNN
 F 3 "~" H 5900 2675 50  0001 C CNN
 	1    5900 2675
@@
 AR Path="/61BFC8AC/61C2038B/61ABA7C0" Ref="#PWR?"  Part="1"
 AR Path="/61BFC8AC/61C20895/61ABA7C0" Ref="#PWR?"  Part="1"
-AR Path="/61C40B21/61ABA7C0" Ref="#PWR?"  Part="1"
+AR Path="/61C40B21/61ABA7C0" Ref="#PWR0143"  Part="1"
 AR Path="/61C417C6/61ABA7C0" Ref="#PWR?"  Part="1"
-AR Path="/61C41B68/61ABA7C0" Ref="#PWR?"  Part="1"
-F 0 "#PWR?" H 5000 5025 50  0001 C CNN
+AR Path="/61C41B68/61ABA7C0" Ref="#PWR0139"  Part="1"
+F 0 "#PWR0143" H 5000 5025 50  0001 C CNN
 F 1 "GND" H 5005 5102 50  0000 C CNN
 F 2 "" H 5000 5275 50  0001 C CNN
@@
 AR Path="/61BFC8AC/61C2038B/61ABA7BF" Ref="#PWR?"  Part="1"
 AR Path="/61BFC8AC/61C20895/61ABA7BF" Ref="#PWR?"  Part="1"
-AR Path="/61C40B21/61ABA7BF" Ref="#PWR?"  Part="1"
+AR Path="/61C40B21/61ABA7BF" Ref="#PWR0144"  Part="1"
 AR Path="/61C417C6/61ABA7BF" Ref="#PWR?"  Part="1"
-AR Path="/61C41B68/61ABA7BF" Ref="#PWR?"  Part="1"
-F 0 "#PWR?" H 5000 1925 50  0001 C CNN
+AR Path="/61C41B68/61ABA7BF" Ref="#PWR0140"  Part="1"
+F 0 "#PWR0144" H 5000 1925 50  0001 C CNN
 F 1 "VCC" H 5015 2248 50  0000 C CNN
 F 2 "" H 5000 2075 50  0001 C CNN
@@
 AR Path="/61BFC8AC/61C20ADE/61ABA7BE" Ref="U?"  Part="1"
 AR Path="/61BFC8AC/61C20AEA/61ABA7BE" Ref="U?"  Part="1"
-AR Path="/61C40B21/61ABA7BE" Ref="U?"  Part="1"
+AR Path="/61C40B21/61ABA7BE" Ref="U11"  Part="1"
 AR Path="/61C417C6/61ABA7BE" Ref="U?"  Part="1"
-AR Path="/61C41B68/61ABA7BE" Ref="U?"  Part="1"
-F 0 "U?" H 5000 3775 50  0000 C CNN
+AR Path="/61C41B68/61ABA7BE" Ref="U10"  Part="1"
+F 0 "U10" H 5000 3775 50  0000 C CNN
 F 1 "8255" H 5000 3675 50  0000 C CNN
 F 2 "Package_DIP:DIP-40_W15.24mm" H 5000 3975 50  0001 C CNN
@@
 P 7875 3375
 AR Path="/61C417C6/61ABA7C4" Ref="C?"  Part="1"
-AR Path="/61C41B68/61ABA7C4" Ref="C?"  Part="1"
-AR Path="/61C40B21/61ABA7C4" Ref="C?"  Part="1"
-F 0 "C?" H 7990 3421 50  0000 L CNN
+AR Path="/61C41B68/61ABA7C4" Ref="C13"  Part="1"
+AR Path="/61C40B21/61ABA7C4" Ref="C14"  Part="1"
+F 0 "C13" H 7990 3421 50  0000 L CNN
 F 1 "100nF" H 7990 3330 50  0000 L CNN
-F 2 "" H 7913 3225 50  0001 C CNN
+F 2 "Capacitor_THT:C_Rect_L4.0mm_W2.5mm_P2.50mm" H 7913 3225 50  0001 C CNN
 F 3 "~" H 7875 3375 50  0001 C CNN
 	1    7875 3375
@@
 P 7875 3225
 AR Path="/61C417C6/61ABA7C5" Ref="#PWR?"  Part="1"
-AR Path="/61C41B68/61ABA7C5" Ref="#PWR?"  Part="1"
-AR Path="/61C40B21/61ABA7C5" Ref="#PWR?"  Part="1"
-F 0 "#PWR?" H 7875 3075 50  0001 C CNN
+AR Path="/61C41B68/61ABA7C5" Ref="#PWR0141"  Part="1"
+AR Path="/61C40B21/61ABA7C5" Ref="#PWR0145"  Part="1"
+F 0 "#PWR0145" H 7875 3075 50  0001 C CNN
 F 1 "VCC" H 7890 3398 50  0000 C CNN
 F 2 "" H 7875 3225 50  0001 C CNN
@@
 P 7875 3525
 AR Path="/61C417C6/61C61024" Ref="#PWR?"  Part="1"
-AR Path="/61C41B68/61C61024" Ref="#PWR?"  Part="1"
-AR Path="/61C40B21/61C61024" Ref="#PWR?"  Part="1"
-F 0 "#PWR?" H 7875 3275 50  0001 C CNN
+AR Path="/61C41B68/61C61024" Ref="#PWR0142"  Part="1"
+AR Path="/61C40B21/61C61024" Ref="#PWR0146"  Part="1"
+F 0 "#PWR0146" H 7875 3275 50  0001 C CNN
 F 1 "GND" H 7880 3352 50  0000 C CNN
 F 2 "" H 7875 3525 50  0001 C CNN
@@
 Text Label 4150 4275 0    50   ~ 0
 D15
+Text Label 4150 3175 0    50   ~ 0
+A1
 Wire Bus Line
 	4050 3000 4050 3175
 Wire Bus Line
 	4050 3675 4050 4500
-Text Label 4150 3175 0    50   ~ 0
-A1
 $EndSCHEMATC

Commit message: assign footprints and edits
Changed lines of the file:
@@
 AR Path="/61C417C6/61ABA7C3" Ref="J?"  Part="1"
 AR Path="/61C41B68/61ABA7C3" Ref="J9"  Part="1"
-F 0 "J9" H 5980 4467 50  0000 L CNN
+F 0 "J12" H 5980 4467 50  0000 L CNN
 F 1 "Conn_01x08" H 5980 4376 50  0000 L CNN
 F 2 "Connector_PinHeader_2.54mm:PinHeader_1x08_P2.54mm_Vertical" H 5900 4475 50  0001 C CNN
@@
 AR Path="/61C417C6/61C3EA07" Ref="J?"  Part="1"
 AR Path="/61C41B68/61C3EA07" Ref="J8"  Part="1"
-F 0 "J8" H 5980 3567 50  0000 L CNN
+F 0 "J11" H 5980 3567 50  0000 L CNN
 F 1 "Conn_01x08" H 5980 3476 50  0000 L CNN
 F 2 "Connector_PinHeader_2.54mm:PinHeader_1x08_P2.54mm_Vertical" H 5900 3575 50  0001 C CNN
@@
 AR Path="/61C417C6/61ABA7C1" Ref="J?"  Part="1"
 AR Path="/61C41B68/61ABA7C1" Ref="J7"  Part="1"
-F 0 "J7" H 5980 2667 50  0000 L CNN
+F 0 "J10" H 5980 2667 50  0000 L CNN
 F 1 "Conn_01x08" H 5980 2576 50  0000 L CNN
 F 2 "Connector_PinHeader_2.54mm:PinHeader_1x08_P2.54mm_Vertical" H 5900 2675 50  0001 C CNN
@@
 AR Path="/61C417C6/61ABA7BE" Ref="U?"  Part="1"
 AR Path="/61C41B68/61ABA7BE" Ref="U10"  Part="1"
-F 0 "U10" H 5000 3775 50  0000 C CNN
+F 0 "U11" H 5000 3775 50  0000 C CNN
 F 1 "8255" H 5000 3675 50  0000 C CNN
 F 2 "Package_DIP:DIP-40_W15.24mm" H 5000 3975 50  0001 C CNN
@@
 AR Path="/61C41B68/61ABA7C4" Ref="C13"  Part="1"
 AR Path="/61C40B21/61ABA7C4" Ref="C14"  Part="1"
-F 0 "C13" H 7990 3421 50  0000 L CNN
+F 0 "C14" H 7990 3421 50  0000 L CNN
 F 1 "100nF" H 7990 3330 50  0000 L CNN
 F 2 "Capacitor_THT:C_Rect_L4.0mm_W2.5mm_P2.50mm" H 7913 3225 50  0001 C CNN

Commit message: begin pcb layout
Parts:
- J10: value Conn_01x08 -> PORT A
- J11: value Conn_01x08 -> PORT B
- J12: value Conn_01x08 -> PORT C
Changed lines of the file:
@@
 AR Path="/61C417C6/61ABA7C3" Ref="J?"  Part="1"
 AR Path="/61C41B68/61ABA7C3" Ref="J9"  Part="1"
-F 0 "J12" H 5980 4467 50  0000 L CNN
-F 1 "Conn_01x08" H 5980 4376 50  0000 L CNN
+F 0 "J9" H 5980 4467 50  0000 L CNN
+F 1 "PORT C" H 5980 4376 50  0000 L CNN
 F 2 "Connector_PinHeader_2.54mm:PinHeader_1x08_P2.54mm_Vertical" H 5900 4475 50  0001 C CNN
 F 3 "~" H 5900 4475 50  0001 C CNN
@@
 AR Path="/61C417C6/61C3EA07" Ref="J?"  Part="1"
 AR Path="/61C41B68/61C3EA07" Ref="J8"  Part="1"
-F 0 "J11" H 5980 3567 50  0000 L CNN
-F 1 "Conn_01x08" H 5980 3476 50  0000 L CNN
+F 0 "J8" H 5980 3567 50  0000 L CNN
+F 1 "PORT B" H 5980 3476 50  0000 L CNN
 F 2 "Connector_PinHeader_2.54mm:PinHeader_1x08_P2.54mm_Vertical" H 5900 3575 50  0001 C CNN
 F 3 "~" H 5900 3575 50  0001 C CNN
@@
 AR Path="/61C417C6/61ABA7C1" Ref="J?"  Part="1"
 AR Path="/61C41B68/61ABA7C1" Ref="J7"  Part="1"
-F 0 "J10" H 5980 2667 50  0000 L CNN
-F 1 "Conn_01x08" H 5980 2576 50  0000 L CNN
+F 0 "J7" H 5980 2667 50  0000 L CNN
+F 1 "PORT A" H 5980 2576 50  0000 L CNN
 F 2 "Connector_PinHeader_2.54mm:PinHeader_1x08_P2.54mm_Vertical" H 5900 2675 50  0001 C CNN
 F 3 "~" H 5900 2675 50  0001 C CNN
@@
 AR Path="/61C417C6/61ABA7C0" Ref="#PWR?"  Part="1"
 AR Path="/61C41B68/61ABA7C0" Ref="#PWR0139"  Part="1"
-F 0 "#PWR0143" H 5000 5025 50  0001 C CNN
+F 0 "#PWR0139" H 5000 5025 50  0001 C CNN
 F 1 "GND" H 5005 5102 50  0000 C CNN
 F 2 "" H 5000 5275 50  0001 C CNN
@@
 AR Path="/61C417C6/61ABA7BF" Ref="#PWR?"  Part="1"
 AR Path="/61C41B68/61ABA7BF" Ref="#PWR0140"  Part="1"
-F 0 "#PWR0144" H 5000 1925 50  0001 C CNN
+F 0 "#PWR0140" H 5000 1925 50  0001 C CNN
 F 1 "VCC" H 5015 2248 50  0000 C CNN
 F 2 "" H 5000 2075 50  0001 C CNN
@@
 AR Path="/61C417C6/61ABA7BE" Ref="U?"  Part="1"
 AR Path="/61C41B68/61ABA7BE" Ref="U10"  Part="1"
-F 0 "U11" H 5000 3775 50  0000 C CNN
+F 0 "U10" H 5000 3775 50  0000 C CNN
 F 1 "8255" H 5000 3675 50  0000 C CNN
 F 2 "Package_DIP:DIP-40_W15.24mm" H 5000 3975 50  0001 C CNN
@@
 AR Path="/61C41B68/61ABA7C4" Ref="C13"  Part="1"
 AR Path="/61C40B21/61ABA7C4" Ref="C14"  Part="1"
-F 0 "C14" H 7990 3421 50  0000 L CNN
+F 0 "C13" H 7990 3421 50  0000 L CNN
 F 1 "100nF" H 7990 3330 50  0000 L CNN
 F 2 "Capacitor_THT:C_Rect_L4.0mm_W2.5mm_P2.50mm" H 7913 3225 50  0001 C CNN
@@
 AR Path="/61C41B68/61ABA7C5" Ref="#PWR0141"  Part="1"
 AR Path="/61C40B21/61ABA7C5" Ref="#PWR0145"  Part="1"
-F 0 "#PWR0145" H 7875 3075 50  0001 C CNN
+F 0 "#PWR0141" H 7875 3075 50  0001 C CNN
 F 1 "VCC" H 7890 3398 50  0000 C CNN
 F 2 "" H 7875 3225 50  0001 C CNN
@@
 AR Path="/61C41B68/61C61024" Ref="#PWR0142"  Part="1"
 AR Path="/61C40B21/61C61024" Ref="#PWR0146"  Part="1"
-F 0 "#PWR0146" H 7875 3275 50  0001 C CNN
+F 0 "#PWR0142" H 7875 3275 50  0001 C CNN
 F 1 "GND" H 7880 3352 50  0000 C CNN
 F 2 "" H 7875 3525 50  0001 C CNN
