File: 8086-system.kicad_pcb (KiCad board)
At the start: 2 copper layers, 184 parts, among them J1 Barrel_Jack +5V, J10 PORT A, J11 PORT B, J12 PORT C, J13 PORT A, J14 PORT B, J15 PORT C, J16 IR4-IR7, J17 Counter0, J18 Counter1, J19 Counter2, J2 Barrel_Jack +12V, J3 ADDRESS BUS, J4 CONTROL BUS, J5 DATA BUS, J6 DSUB-9, J7 PORT A, J8 PORT B, J9 PORT C, SW1 RESET, SW10 C1,R3, SW11 C2,R0, SW12 C2,R1, SW13 C2,R2, SW14 C2,R3, SW15 C3,R0, SW16 C3,R1, SW17 C3,R2, SW18 C3,R3, SW19 C4,R0, SW2 IR0, SW20 C4,R1, SW21 C4,R2, SW22 C4,R3, SW23 SHIFT, SW24 CNTL, SW25 NMI, SW26 SW_DIP_x08, SW3 C0,R0, SW4 C0,R1, SW5 C0,R2, SW6 C0,R3, SW7 C1,R0, SW8 C1,R1, SW9 C1,R2, U1 8284, U10 8255, U11 8255, U12 8255, U13 8259, U14 74LS14, U15 pkd8279, U16 74LS138, U17 8254, U18 8086_Min_Mode, U19 74LS374, U2 16550, U20 74LS244, U21 74LS374, U22 74LS374, U23 74LS245, U24 74LS245, U25 74LS138, U26 74LS138, U27 28F010, U28 28F010, U29 74LS30, U3 max235cpg, U30 PAL16L8, U31 PAL16L8, U32 74LS02, U33 74LS32, U34 74LS374, U36 74LS374, U37 HDSP-A153, U38 74LS374, U39 74LS244, U4 74LS138, U40 HDSP-A153, U5 74LS138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

Commit message: Layout PPI, interrupt, counter, and UART blocks
Parts:
- moved SW2 889.9 mm to (448.3, 664.2)
- moved R7 556.5 mm to (450.9, 656.6), turned to 180 degrees
- moved R9 550.7 mm to (450.9, 649.0), turned to 180 degrees
- moved R10 547.8 mm to (450.9, 645.2), turned to 180 degrees
- moved R8 539.9 mm to (440.7, 652.8), turned to 0 degrees
- moved C17 536.8 mm to (409.6, 638.2)
- moved U13 536.8 mm to (400.7, 644.5)
- moved R6 534.7 mm to (420.4, 678.2), turned to 90 degrees
- moved R4 533.4 mm to (424.2, 678.2), turned to 0 degrees
- moved J16 531.4 mm to (434.3, 647.1)
- moved U10 529.4 mm to (638.8, 549.9), turned to 180 degrees
- moved R5 522.8 mm to (424.2, 673.1), turned to 0 degrees
- moved D2 520.0 mm to (434.3, 660.4), turned to 270 degrees
- moved U14 517.0 mm to (428.0, 660.4), turned to 180 degrees
- moved C16 515.8 mm to (428.0, 666.8), turned to 180 degrees
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Routing:
- net Net-(J15-Pad3): track 56.4 -> 5.94 mm
- net Net-(J15-Pad2): track 51.0 -> 5.94 mm
- net Net-(J17-Pad2): track 0.00 -> 43.3 mm
- net Net-(J15-Pad4): track 53.9 -> 12.9 mm
- net Net-(J15-Pad1): track 52.9 -> 13.0 mm
- net Net-(J15-Pad5): track 42.7 -> 4.89 mm
- net Net-(U2-Pad10): track 0.00 -> 37.7 mm
- net Net-(U2-Pad11): track 0.00 -> 37.7 mm
- net Net-(J17-Pad1): track 0.00 -> 36.6 mm
- net Net-(U2-Pad37): track 0.00 -> 35.5 mm
- net Net-(J6-Pad9): track 0.00 -> 35.1 mm
- net Net-(U2-Pad38): track 0.00 -> 34.4 mm
- net Net-(J15-Pad6): track 39.1 -> 4.89 mm
- net Net-(J15-Pad7): track 36.2 -> 4.89 mm
- net Net-(J15-Pad8): track 34.3 -> 4.89 mm
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Other:
- copper layers 2 -> 4

Commit message: more traces routed
Parts:
- moved SW2 667.0 mm to (85.5, 104.5)
- moved J1 489.2 mm to (80.5, 223.0), turned to 90 degrees
- moved R23 487.3 mm to (72.9, 205.2), turned to 270 degrees
- moved C1 482.5 mm to (81.8, 215.4), turned to 180 degrees
- moved J2 478.9 mm to (96.5, 223.0), turned to 90 degrees
- moved D12 475.2 mm to (81.8, 204.0), turned to 180 degrees
- moved C2 472.6 mm to (97.8, 215.4), turned to 180 degrees
- moved U31 450.9 mm to (124.2, 59.2)
- moved U30 450.8 mm to (141.5, 59.2)
- moved J16 437.5 mm to (346.6, 218.4)
- moved C16 437.5 mm to (340.2, 238.1)
- moved D2 437.5 mm to (346.6, 231.8)
- moved R10 437.5 mm to (363.1, 216.5)
- moved R5 437.5 mm to (336.4, 244.5)
- moved R7 437.5 mm to (363.1, 228.0)
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Connections:
- D13 pad 1: /8279-keyboard/CL1 -> Net-(D13-Pad1)
- SW3 pad 2: /8279-keyboard/CL1 -> Net-(D13-Pad1)
Routing:
- net /8086-processor/D0: track 0.00 -> 405.0 mm
- net /RESET: track 0.00 -> 399.8 mm, vias 0 -> 1
- net /8086-processor/D1: track 0.00 -> 392.3 mm
- net Net-(D2-Pad2): track 18.3 -> 404.9 mm
- net /8086-processor/D7: track 0.00 -> 386.4 mm
- net /8086-processor/D6: track 0.00 -> 382.0 mm
- net /8086-processor/D2: track 0.00 -> 381.0 mm
- net /8086-processor/A1: track 0.00 -> 376.9 mm
- net /8086-processor/D3: track 0.00 -> 375.5 mm
- net /8086-processor/D5: track 0.00 -> 372.9 mm
- net /8086-processor/D4: track 0.00 -> 367.3 mm
- net /~RD: track 0.00 -> 345.3 mm
- net /KEYBOARD_INTR: track 0.00 -> 333.4 mm
- net /~WR: track 0.00 -> 319.7 mm, vias 0 -> 1
- net /8086-processor/A0: track 0.00 -> 306.2 mm
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- added copper zone on In2.Cu, net GND
- added copper zone on In1.Cu, net VCC
Other:
- board outline added: 391.2 x 237.5 mm
- net class +12V added: clearance 0.2, trace_width 0.5, via_dia 0.8, via_drill 0.4

Commit message: Route some more, starting re-doing memory routing
Parts:
- U25, U26: footprint Package_DIP:DIP-20_W7.62mm -> Package_DIP:DIP-16_W7.62mm
- moved U27 360.6 mm to (557.4, 152.4)
- moved U28 360.6 mm to (534.5, 152.4)
- moved U7 353.0 mm to (596.8, 148.0)
- moved U8 353.0 mm to (584.1, 148.0)
- moved U9 353.0 mm to (571.4, 148.0)
- moved U6 353.0 mm to (609.5, 148.0)
- moved C14 37.2 mm to (400.1, 129.5)
- moved C13 35.8 mm to (400.1, 194.9)
- moved C15 34.0 mm to (400.1, 64.8)
- moved C7 26.0 mm to (243.7, 99.1)
- moved C9 26.0 mm to (269.1, 99.1)
- moved C1 21.6 mm to (81.8, 237.0)
- moved C2 21.6 mm to (97.8, 237.0)
- moved D12 21.6 mm to (81.8, 225.6)
- moved J1 21.6 mm to (80.5, 244.6)
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Routing:
- net /clock-generator/~RES: track 23.3 -> 297.3 mm, vias 0 -> 2
- net /8086-processor/A12: track 140.4 -> 389.0 mm, vias 0 -> 6
- net /8086-processor/A11: track 151.6 -> 395.2 mm, vias 0 -> 6
- net /8086-processor/A15: track 201.5 -> 444.9 mm, vias 1 -> 6
- net /8086-processor/A1: track 376.9 -> 592.5 mm, vias 0 -> 7
- net /8086-processor/A13: track 170.6 -> 383.3 mm, vias 0 -> 6
- net /8086-processor/A14: track 212.2 -> 424.6 mm, vias 1 -> 6
- net /8086-processor/D15: track 184.9 -> 390.5 mm, vias 0 -> 4
- net /8086-processor/A10: track 145.1 -> 349.2 mm, vias 0 -> 6
- net /8086-processor/D14: track 192.1 -> 381.3 mm, vias 0 -> 4
- net /8086-processor/A9: track 138.9 -> 326.4 mm, vias 0 -> 6
- net /8086-processor/D13: track 195.2 -> 375.5 mm, vias 0 -> 4
- net /8086-processor/D7: track 386.4 -> 561.1 mm, vias 0 -> 3
- net /8086-processor/D6: track 382.0 -> 547.4 mm, vias 0 -> 3
- net /8086-processor/D5: track 372.9 -> 534.6 mm, vias 0 -> 3
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
Commit message: continued pcb routing
Parts:
- moved U6 295.2 mm to (324.7, 70.0), turned to 270 degrees
- moved U7 279.8 mm to (324.7, 82.7), turned to 270 degrees
- moved U8 264.6 mm to (324.7, 95.4), turned to 270 degrees
- moved U9 249.8 mm to (324.7, 108.1), turned to 270 degrees
- moved C33 243.9 mm to (394.8, 143.8), turned to 270 degrees
- moved U27 230.2 mm to (329.2, 122.0), turned to 270 degrees
- moved C34 215.3 mm to (394.8, 128.3), turned to 270 degrees
- moved U26 208.2 mm to (370.0, 148.9), turned to 90 degrees
- moved U28 205.5 mm to (329.2, 144.9), turned to 270 degrees
- moved U25 179.7 mm to (370.0, 133.4), turned to 90 degrees
- moved C31 176.8 mm to (329.1, 163.4), turned to 180 degrees
- moved C29 155.7 mm to (329.2, 141.2), turned to 180 degrees
- moved C11 141.8 mm to (387.6, 95.0), turned to 270 degrees
- moved J3 114.5 mm to (360.6, 135.9)
- moved C12 112.9 mm to (388.1, 79.0), turned to 270 degrees
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Routing:
- net /8086-processor/A0: track 306.2 -> 18.2 mm
- net /~BHE: track 199.6 -> 18.2 mm
- net /8086-processor/A18: track 292.3 -> 138.2 mm, vias 0 -> 1
- net /8086-processor/A19: track 290.9 -> 141.0 mm
- net +12V: track 182.7 -> 313.1 mm
- net /8086-processor/D10: track 369.6 -> 488.3 mm, vias 4 -> 5
- net /8086-processor/D8: track 377.3 -> 496.0 mm, vias 5 -> 6
- net /8086-processor/D9: track 371.3 -> 488.9 mm, vias 5 -> 6
- net /8086-processor/D15: track 390.5 -> 498.3 mm, vias 4 -> 5
- net /8086-processor/D14: track 381.3 -> 489.0 mm, vias 4 -> 5
- net /8086-processor/D13: track 375.5 -> 482.3 mm, vias 4 -> 5
- net /8086-processor/D12: track 366.2 -> 472.5 mm, vias 4 -> 5
- net /8086-processor/D11: track 366.5 -> 472.4 mm, vias 4 -> 5
- net /8086-processor/D0: track 552.3 -> 647.3 mm, vias 3 -> 4
- net /8086-processor/D1: track 537.1 -> 631.8 mm, vias 3 -> 4
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Other:
- board size 391.2 x 237.5 mm -> 391.2 x 255.5 mm

Commit message: Route data bus lines, most chip selects
Parts:
- moved J2 235.1 mm to (196.8, 73.9), turned to 270 degrees
- moved C2 219.7 mm to (195.6, 81.5), turned to 0 degrees
- moved J5 163.3 mm to (210.2, 89.5)
- moved U29 162.4 mm to (368.9, 80.0), turned to 270 degrees
- moved U30 152.4 mm to (373.9, 95.0)
- moved U31 152.4 mm to (356.6, 95.0)
- moved C36 150.4 mm to (379.1, 127.6)
- moved C35 140.0 mm to (351.8, 114.9), turned to 270 degrees
- moved J3 79.0 mm to (318.1, 69.2)
- moved U25 54.1 mm to (316.0, 136.6)
- moved U26 54.1 mm to (316.0, 152.0)
- moved C33 54.1 mm to (340.8, 147.0)
- moved C34 54.1 mm to (340.8, 131.5)
- moved RN2 52.6 mm to (301.0, 219.7), turned to 270 degrees
- moved C11 52.0 mm to (340.6, 117.2)
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Connections:
- SW26 pad 10: Net-(RN2-Pad10) -> Net-(RN2-Pad15)
- SW26 pad 11: Net-(RN2-Pad11) -> Net-(RN2-Pad14)
- SW26 pad 12: Net-(RN2-Pad12) -> Net-(RN2-Pad13)
- SW26 pad 13: Net-(RN2-Pad13) -> Net-(RN2-Pad12)
- SW26 pad 14: Net-(RN2-Pad14) -> Net-(RN2-Pad11)
- SW26 pad 15: Net-(RN2-Pad15) -> Net-(RN2-Pad10)
- SW26 pad 16: Net-(RN2-Pad16) -> Net-(RN2-Pad9)
- SW26 pad 9: Net-(RN2-Pad9) -> Net-(RN2-Pad16)
- U30 pad 18: /~CS_PPI2 -> /~CS_PPI1
- U30 pad 19: /~CS_PPI1 -> /~CS_PPI2
- U31 pad 17: /~LED_CS -> /~ODD_7_SEG_CS
- U31 pad 18: /~ODD_7_SEG_CS -> /~EVEN_7_SEG_CS
- U31 pad 19: /~EVEN_7_SEG_CS -> /~LED_CS
- U39 pad 11: Net-(RN2-Pad12) -> Net-(RN2-Pad13)
- U39 pad 13: Net-(RN2-Pad11) -> Net-(RN2-Pad14)
- U39 pad 15: Net-(RN2-Pad10) -> Net-(RN2-Pad15)
- U39 pad 17: Net-(RN2-Pad9) -> Net-(RN2-Pad16)
- U39 pad 2: Net-(RN2-Pad16) -> Net-(RN2-Pad9)
- U39 pad 4: Net-(RN2-Pad15) -> Net-(RN2-Pad10)
- U39 pad 6: Net-(RN2-Pad14) -> Net-(RN2-Pad11)
- U39 pad 8: Net-(RN2-Pad13) -> Net-(RN2-Pad12)
Routing:
- net /8086-processor/A2: track 372.0 -> 706.1 mm, vias 7 -> 6
- net /clock-generator/~RES: track 297.3 -> 23.3 mm, vias 2 -> 0
- net Net-(D3-Pad1): track 298.6 -> 62.2 mm, vias 3 -> 0
- net /~CS_COUNTER: track 0.00 -> 224.5 mm
- net /8086-processor/A1: track 573.8 -> 793.6 mm, vias 8 -> 6
- net /~CS_PPI3: track 0.00 -> 209.9 mm
- net /~CS_INTR: track 0.00 -> 180.3 mm
- net /~LED_CS: track 31.4 -> 206.9 mm, vias 1 -> 0
- net +12V: track 313.1 -> 147.2 mm
- net /~EVEN_7_SEG_CS: track 43.2 -> 208.2 mm
- net /~ODD_7_SEG_CS: track 48.3 -> 206.5 mm
- net /~LCD_CS: track 43.7 -> 196.3 mm
- net /~CS_PPI1: track 0.00 -> 145.4 mm
- net /8086-processor/A3: track 270.0 -> 394.5 mm, vias 7 -> 6
- net /~CS_KEYBOARD: track 120.1 -> 0.00 mm, vias 1 -> 0
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