File: 8086-system.kicad_pcb (KiCad board)
At the start: 4 copper layers, 391.2 x 255.5 mm, 184 parts, among them J1 Barrel_Jack +5V, J10 PORT A, J11 PORT B, J12 PORT C, J13 PORT A, J14 PORT B, J15 PORT C, J16 IR4-IR7, J17 Counter0, J18 Counter1, J19 Counter2, J2 Barrel_Jack +12V, J3 ADDRESS BUS, J4 CONTROL BUS, J5 DATA BUS, J6 DSUB-9, J7 PORT A, J8 PORT B, J9 PORT C, SW1 RESET, SW10 C1,R3, SW11 C2,R0, SW12 C2,R1, SW13 C2,R2, SW14 C2,R3, SW15 C3,R0, SW16 C3,R1, SW17 C3,R2, SW18 C3,R3, SW19 C4,R0, SW2 IR0, SW20 C4,R1, SW21 C4,R2, SW22 C4,R3, SW23 SHIFT, SW24 CNTL, SW25 NMI, SW26 SW_DIP_x08, SW3 C0,R0, SW4 C0,R1, SW5 C0,R2, SW6 C0,R3, SW7 C1,R0, SW8 C1,R1, SW9 C1,R2, U1 8284, U10 8255, U11 8255, U12 8255, U13 8259, U14 74LS14, U15 pkd8279, U16 74LS138, U17 8254, U18 8086_Min_Mode, U19 74LS374, U2 16550, U20 74LS244, U21 74LS374, U22 74LS374, U23 74LS245, U24 74LS245, U25 74LS138, U26 74LS138, U27 28F010, U28 28F010, U29 74LS30, U3 max235cpg, U30 PAL16L8, U31 PAL16L8, U32 74LS02, U33 74LS32, U34 74LS374, U36 74LS374, U37 HDSP-A153, U38 74LS374, U39 74LS244, U4 74LS138, U40 HDSP-A153, U5 74LS138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

Commit message: more pcb routing
Parts:
- moved C22 5.34 mm to (317.8, 175.8), turned to 270 degrees
- moved C24 5.02 mm to (342.1, 171.2), turned to 270 degrees
- moved C25 4.77 mm to (340.9, 208.9)
- moved R3 3.24 mm to (439.8, 89.2)
- moved C23 3.12 mm to (326.8, 241.7)
- moved C26 1.66 mm to (357.5, 178.4)
Routing:
- net /~WR: track 284.6 -> 843.8 mm, vias 0 -> 3
- net /~RD: track 364.3 -> 904.8 mm, vias 0 -> 1
- net /8086-processor/A1: track 793.6 -> 1078.2 mm, vias 6 -> 8
- net /UART_INTR: track 0.00 -> 225.0 mm, vias 0 -> 2
- net /8086-processor/A2: track 706.1 -> 913.3 mm, vias 6 -> 8
- net /8086-processor/D0: track 636.5 -> 842.5 mm, vias 7 -> 8
- net /8086-processor/D1: track 640.6 -> 845.3 mm
- net /8086-processor/D2: track 648.4 -> 852.0 mm
- net /8086-processor/D3: track 616.1 -> 819.6 mm
- net /8086-processor/D4: track 660.1 -> 861.4 mm
- net /8086-processor/D7: track 677.6 -> 878.6 mm
- net /8086-processor/D5: track 675.0 -> 875.2 mm
- net /RESET: track 523.9 -> 724.1 mm, vias 2 -> 5
- net /8086-processor/D6: track 685.3 -> 884.4 mm
- net /8086-processor/A18: track 33.5 -> 180.7 mm
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